Commit message: wip bullet loadURDF flag: dynamics parameters from URDF file

File: description/indy7.urdf (robot description, URDF)
Before this commit: robot indy7, 9 links, 8 joints
Links:
- removed link base_link
- removed link forearm_link
- removed link shoulder_link
- removed link upper_arm_link
- removed link wrist_1_link
- removed link wrist_2_link
- removed link wrist_3_link
- added link link0, mass 1.59306955; collision cylinder length=0.075 radius=0.102; visual mesh filename=meshes/stl/Indy7_0.stl
- added link link1, mass 11.8030102; collision cylinder length=0.109 radius=0.075; collision cylinder length=0.222 radius=0.075
- added link link2, mass 7.99292141; collision cylinder length=0.09 radius=0.075; collision cylinder length=0.1205 radius=0.045
- added link link3, mass 2.99134127; collision cylinder length=0.075 radius=0.045; collision cylinder length=0.267 radius=0.045
- added link link4, mass 2.12317035; collision cylinder length=0.083 radius=0.045; collision cylinder length=0.114 radius=0.045
- added link link5, mass 2.28865091; collision cylinder length=0.069 radius=0.045; collision cylinder length=0.168 radius=0.045
- added link link6, mass 0.40083918; collision cylinder length=0.06 radius=0.045; visual mesh filename=meshes/stl/Indy7_6.stl
- link tcp: mass 0.0000 -> 0.000001; geometry 
Joints:
- removed joint tcp_joint
- added joint indy7_tcp: type fixed, parent link6, child tcp, origin xyz=0 0 0.06 rpy=0 0 0
- joint joint0: child shoulder_link -> link1; limit lower=-3.05432619099 upper=3.05432619099 effort=50 velocity=1 -> lower=-3.0543261909900763 upper=3.0543261909900763 effort=10 velocity=1; parent base_link -> link0
- joint joint1: child upper_arm_link -> link2; limit lower=-3.05432619099 upper=3.05432619099 effort=50 velocity=1 -> lower=-3.0543261909900763 upper=3.0543261909900763 effort=10 velocity=1; origin xyz=0 -0.10900000 0.22200000 rpy=1.57079632679 1.57079632679 0 -> xyz=0 -0.10900000 0.22200000 rpy=1.5707963267948966 1.5707963267948966 0; parent shoulder_link -> link1
- joint joint2: child forearm_link -> link3; limit lower=-3.05432619099 upper=3.05432619099 effort=50 velocity=1 -> lower=-3.0543261909900763 upper=3.0543261909900763 effort=10 velocity=1; parent upper_arm_link -> link2
- joint joint3: child wrist_1_link -> link4; limit lower=-3.05432619099 upper=3.05432619099 effort=50 velocity=1 -> lower=-3.0543261909900763 upper=3.0543261909900763 effort=10 velocity=1; origin xyz=-0.26700000 +0.00000000 -0.07500000 rpy=-1.57079632679 0 1.57079632679 -> xyz=-0.26700000 +0.00000000 -0.07500000 rpy=-1.5707963267948966 0 1.5707963267948966; parent forearm_link -> link3
- joint joint4: child wrist_2_link -> link5; limit lower=-3.05432619099 upper=3.05432619099 effort=50 velocity=1 -> lower=-3.0543261909900763 upper=3.0543261909900763 effort=10 velocity=1; origin xyz=+0.00000000 -0.11400000 +0.08300000 rpy=1.57079632679 1.57079632679 0 -> xyz=+0.00000000 -0.11400000 +0.08300000 rpy=1.5707963267948966 1.5707963267948966 0; parent wrist_1_link -> link4
- joint joint5: child wrist_3_link -> link6; limit lower=-3.75245789179 upper=3.75245789179 effort=50 velocity=1 -> lower=-3.752457891787808 upper=3.752457891787808 effort=10 velocity=1; origin xyz=-0.16800000 +0.00000000 +0.06900000 rpy=-1.57079632679 0 1.57079632679 -> xyz=-0.16800000 +0.00000000 +0.06900000 rpy=-1.5707963267948966 0 1.5707963267948966; parent wrist_2_link -> link5
- joint world_joint: child base_link -> link0

Commit message: update

File: description/indy7.urdf (robot description, URDF)
Before this commit: robot indy7, 9 links, 8 joints
Links:
- removed link world
- link link0: mass 1.59306955 -> 1.67030785; geometry visual mesh filename=meshes/stl/Indy7_0.stl
- link link1: mass 11.8030102 -> 11.44444535; geometry visual mesh filename=meshes/stl/Indy7_1.stl
- link link2: mass 7.99292141 -> 5.84766553; geometry visual mesh filename=meshes/stl/Indy7_2.stl
- link link3: mass 2.99134127 -> 2.68206064; geometry visual mesh filename=meshes/stl/Indy7_3.stl
- link link4: mass 2.12317035 -> 2.12987371; geometry visual mesh filename=meshes/stl/Indy7_4.stl
- link link5: mass 2.28865091 -> 2.22412271; geometry visual mesh filename=meshes/stl/Indy7_5.stl
- link link6: mass 0.40083918 -> 0.38254932; geometry visual mesh filename=meshes/stl/Indy7_6.stl
Joints:
- removed joint world_joint
- joint indy7_tcp: origin xyz=0 0 0.06 rpy=0 0 0 -> xyz=0 0 0.0795 rpy=0 0 0

Commit message: update

File: description/indy7.urdf (robot description, URDF)
Before this commit: robot indy7, 8 links, 7 joints
Links:
- link link0: geometry visual mesh filename=meshes/stl/indy7/Indy7_0.stl
- link link1: geometry visual mesh filename=meshes/stl/indy7/indy7_1.stl
- link link2: geometry visual mesh filename=meshes/stl/indy7/indy7_2.stl
- link link3: geometry visual mesh filename=meshes/stl/indy7/indy7_3.stl
- link link4: geometry visual mesh filename=meshes/stl/indy7/indy7_4.stl
- link link5: geometry visual mesh filename=meshes/stl/indy7/indy7_5.stl
- link link6: geometry visual mesh filename=meshes/stl/indy7/indy7_6.stl

File: description/indyrp2.urdf (robot description, URDF)
Before this commit: robot indyrp2, 9 links, 8 joints
Links:
- link link0: geometry visual mesh filename=meshes/stl/indyrp2/IndyRP2_0.stl
- link link1: geometry visual mesh filename=meshes/stl/indyrp2/IndyRP2_1.stl
- link link2: geometry visual mesh filename=meshes/stl/indyrp2/IndyRP2_2.stl
- link link3: geometry visual mesh filename=meshes/stl/indyrp2/IndyRP2_3.stl
- link link4: geometry visual mesh filename=meshes/stl/indyrp2/IndyRP2_4.stl
- link link5: geometry visual mesh filename=meshes/stl/indyrp2/IndyRP2_5.stl
- link link6: geometry visual mesh filename=meshes/stl/indyrp2/IndyRP2_6.stl
- link link7: geometry visual mesh filename=meshes/stl/indyrp2/IndyRP2_7.stl
